File: GameBoy-DMG-Buttons.sch (EAGLE design)
At the start: 13 parts

Commit message: Minor updates on the schematic
Parts:
- A, B, DOWN, LEFT, RIGHT, UP, X, Y: value BUTTON_PAD_6MM -> Pad 6mm
- SELECT, SELECT2, START, START2: value BUTTON_PAD_4MM -> Pad 4mm
Other:
- note added: "DMG Button Breakout"
- note added: "JRodrigo.net"
- note added: "Licenced under Creative Commons - Attribution and Share Alike by J.Rodrigo"
- moved on the sheet: A, B, CON, DOWN, LEFT, RIGHT, SELECT, SELECT2, START, START2, UP, X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
