File: GameBoy-DMG-Buttons.brd (EAGLE design)
At the start: 81.5 x 52 mm, 13 parts

Commit message: Silkscreen fixed
Parts:
- A, B, DOWN, LEFT, RIGHT, UP, X, Y: value BUTTON_PAD_6MM -> Pad 6mm
- SELECT, SELECT2, START, START2: value BUTTON_PAD_4MM -> Pad 4mm
Changed lines of the file:
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@@
 <setting verticaltext="up"/>
 </settings>
-<grid distance="25" unitdist="mil" unit="mil" style="lines" multiple="1" display="yes" altdistance="0.025" altunitdist="inch" altunit="inch"/>
+<grid distance="25" unitdist="mil" unit="mm" style="lines" multiple="1" display="yes" altdistance="0.025" altunitdist="inch" altunit="inch"/>
 <layers>
 <layer number="1" name="Top" color="4" fill="1" visible="yes" active="yes"/>
@@
 <wire x1="55.88" y1="38.1" x2="63.5" y2="25.4" width="3.81" layer="22"/>
 <wire x1="62.23" y1="41.91" x2="69.85" y2="29.21" width="3.81" layer="22"/>
-<polygon width="0.4064" layer="22">
-<vertex x="68.58" y="52.07" curve="25"/>
-<vertex x="67.31" y="45.72"/>
-<vertex x="67.31" y="44.45" curve="90"/>
-<vertex x="78.74" y="33.02"/>
-<vertex x="81.28" y="33.02"/>
-<vertex x="81.28" y="43.18" curve="90"/>
-<vertex x="72.39" y="52.07"/>
-<vertex x="73.66" y="52.07"/>
-</polygon>
 <wire x1="30.5" y1="38.5" x2="29" y2="35.25" width="0.5" layer="22" curve="-230.194429"/>
 <wire x1="30.5" y1="38.5" x2="29" y2="35.25" width="0.5" layer="22" curve="-230.194429"/>
+<polygon width="0.4064" layer="22">
+<vertex x="81.5" y="31.75"/>
+<vertex x="81.5" y="43.18" curve="90"/>
+<vertex x="72.39" y="52"/>
+<vertex x="67.31" y="52" curve="110"/>
+</polygon>
 </plain>
 <attributes>
@@
 <elements>
 <element name="CON" library="pinhead" package="1X11" value="" x="28.375" y="45.165"/>
-<element name="UP" library="jrodrigo" package="BUTTON_PAD-D6MM" value="BUTTON_PAD_6MM" x="14.75" y="36.35"/>
-<element name="DOWN" library="jrodrigo" package="BUTTON_PAD-D6MM" value="BUTTON_PAD_6MM" x="14.75" y="18"/>
-<element name="LEFT" library="jrodrigo" package="BUTTON_PAD-D6MM" value="BUTTON_PAD_6MM" x="5.55" y="27.15"/>
-<element name="RIGHT" library="jrodrigo" package="BUTTON_PAD-D6MM" value="BUTTON_PAD_6MM" x="23.85" y="27.15" rot="R180"/>
-<element name="B" library="jrodrigo" package="BUTTON_PAD-D6MM" value="BUTTON_PAD_6MM" x="58.65" y="25.15"/>
-<element name="A" library="jrodrigo" package="BUTTON_PAD-D6MM" value="BUTTON_PAD_6MM" x="73.15" y="32"/>
-<element name="Y" library="jrodrigo" package="BUTTON_PAD-D6MM" value="BUTTON_PAD_6MM" x="52.35" y="39.85"/>
-<element name="X" library="jrodrigo" package="BUTTON_PAD-D6MM" value="BUTTON_PAD_6MM" x="66.85" y="46.7"/>
-<element name="SELECT" library="jrodrigo" package="BUTTON_PAD-D4MM" value="BUTTON_PAD_4MM" x="31.4" y="6.75" rot="R207"/>
-<element name="START" library="jrodrigo" package="BUTTON_PAD-D4MM" value="BUTTON_PAD_4MM" x="46.65" y="6.75" rot="R27"/>
-<element name="SELECT2" library="jrodrigo" package="BUTTON_PAD-D4MM" value="BUTTON_PAD_4MM" x="26" y="3.95" rot="R27"/>
-<element name="START2" library="jrodrigo" package="BUTTON_PAD-D4MM" value="BUTTON_PAD_4MM" x="41.25" y="3.95" rot="R207"/>
+<element name="UP" library="jrodrigo" package="BUTTON_PAD-D6MM" value="Pad 6mm" x="14.75" y="36.35"/>
+<element name="DOWN" library="jrodrigo" package="BUTTON_PAD-D6MM" value="Pad 6mm" x="14.75" y="18"/>
+<element name="LEFT" library="jrodrigo" package="BUTTON_PAD-D6MM" value="Pad 6mm" x="5.55" y="27.15"/>
+<element name="RIGHT" library="jrodrigo" package="BUTTON_PAD-D6MM" value="Pad 6mm" x="23.85" y="27.15" rot="R180"/>
+<element name="B" library="jrodrigo" package="BUTTON_PAD-D6MM" value="Pad 6mm" x="58.65" y="25.15"/>
+<element name="A" library="jrodrigo" package="BUTTON_PAD-D6MM" value="Pad 6mm" x="73.15" y="32"/>
+<element name="Y" library="jrodrigo" package="BUTTON_PAD-D6MM" value="Pad 6mm" x="52.35" y="39.85"/>
+<element name="X" library="jrodrigo" package="BUTTON_PAD-D6MM" value="Pad 6mm" x="66.85" y="46.7"/>
+<element name="SELECT" library="jrodrigo" package="BUTTON_PAD-D4MM" value="Pad 4mm" x="31.4" y="6.75" rot="R207"/>
+<element name="START" library="jrodrigo" package="BUTTON_PAD-D4MM" value="Pad 4mm" x="46.65" y="6.75" rot="R27"/>
+<element name="SELECT2" library="jrodrigo" package="BUTTON_PAD-D4MM" value="Pad 4mm" x="26" y="3.95" rot="R27"/>
+<element name="START2" library="jrodrigo" package="BUTTON_PAD-D4MM" value="Pad 4mm" x="41.25" y="3.95" rot="R207"/>
 </elements>
 <signals>
